File: Casualty6.kicad_pcb (KiCad board)
At the start: 2 copper layers, 80 x 54.5 mm, 91 parts, among them J1 9V, J2 G, J3 IN/LED/GND/OUT, J4 IG, J5 OG, SW1 DPDT, SW2 DPDT, U1 LM13700, U2 LM13700, U3 TL072, U4 TL072, U5 TL072, U6 TL072

Commit message: Casualty 6: REGEN fix (U5B non-inverting summer, R48-R50) from ngspice sim; slotted DPDT toggle footprint; full re-route (DRC 0); sim scripts and notes
Co-Authored-By: Claude Opus 5.5 <noreply@anthropic.com>
Parts:
- added R48: 10k, Resistor_SMD:R_0805_2012Metric_Pad1.20x1.40mm_HandSolder, F.Cu at (188.0, 100.1)
- added R49: 6k8, Resistor_SMD:R_0805_2012Metric_Pad1.20x1.40mm_HandSolder, F.Cu at (180.0, 95.3)
- added R50: 10k, Resistor_SMD:R_0805_2012Metric_Pad1.20x1.40mm_HandSolder, F.Cu at (183.8, 97.3)
Connections:
- C6 pad 1: /DRY -> /X
- R27 pad 1: /DRY -> /X
- R30 pad 2: /REGEN_IN -> /REGEN_SUM
- RV6 pad 3: /DRY -> /X
- U5 pad 5: /VREF -> /REGEN_SUM
- U5 pad 7: Net-(U5B--) -> /X
Routing:
- net /X: track 0.00 -> 80.1 mm, vias 0 -> 1
- net /REGEN_SUM: track 0.00 -> 52.4 mm, vias 0 -> 3
- net Net-(RV3-Pad2): track 65.4 -> 110.2 mm, vias 0 -> 2
- net /DRY: track 14.9 -> 57.4 mm, vias 0 -> 2
- net Net-(SW1B-A): track 101.1 -> 62.3 mm, vias 2 -> 3
- net /VREF: track 202.3 -> 179.2 mm, vias 4 -> 7
- net Net-(C2-Pad2): track 21.9 -> 41.2 mm
- net Net-(U2A--): track 20.6 -> 36.7 mm, vias 3 -> 0
- net Net-(SW2A-B): track 31.9 -> 45.8 mm, vias 2 -> 1
- net GND: track 352.8 -> 338.9 mm, vias 3 -> 5
- net Net-(R34-Pad1): track 16.9 -> 30.0 mm, vias 1 -> 0
- net +9V: track 224.7 -> 237.5 mm, vias 8 -> 6
- net Net-(SW1A-A): track 46.8 -> 38.6 mm
- net Net-(U6B--): track 42.1 -> 34.2 mm, vias 1 -> 3
- net Net-(SW2B-A): track 59.4 -> 67.2 mm
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
Commit message: Casualty 6: CV IN (J6 + R51 10k) and LFO OUT (J7 + R52 1k) pads; full re-route (DRC 0)
Co-Authored-By: Claude Opus 5.5 <noreply@anthropic.com>
Parts:
- added J6: CV IN, Connector_Wire:SolderWire-0.5sqmm_1x01_D0.9mm_OD2.1mm, F.Cu at (112.5, 102.5)
- added J7: LFO OUT, Connector_Wire:SolderWire-0.5sqmm_1x01_D0.9mm_OD2.1mm, F.Cu at (112.5, 114.0)
- added R51: 10k, Resistor_SMD:R_0805_2012Metric_Pad1.20x1.40mm_HandSolder, F.Cu at (116.0, 102.5)
- added R52: 1k, Resistor_SMD:R_0805_2012Metric_Pad1.20x1.40mm_HandSolder, F.Cu at (167.8, 114.9)
Routing:
- net /LFO_OUT: track 0.00 -> 73.4 mm, vias 0 -> 1
- net Net-(R52-Pad1): track 110.2 -> 70.0 mm, vias 2 -> 1
- net GND: track 338.9 -> 362.1 mm
- net +9V: track 237.5 -> 260.4 mm, vias 6 -> 13
- net /DRY: track 57.4 -> 79.5 mm
- net Net-(U2A--): track 36.7 -> 18.8 mm
- net Net-(C2-Pad2): track 41.2 -> 23.7 mm
- net Net-(R34-Pad1): track 30.0 -> 17.0 mm, vias 0 -> 1
- net /CV: track 59.1 -> 71.9 mm, vias 2 -> 1
- net Net-(SW1B-B): track 40.5 -> 52.9 mm
- net Net-(SW2A-B): track 45.8 -> 34.1 mm, vias 1 -> 0
- net Net-(SW2B-A): track 67.2 -> 78.5 mm, vias 3 -> 2
- net /PHASE_OUT: track 68.5 -> 59.3 mm, vias 3 -> 4
- net /REGEN_IN: track 19.6 -> 11.5 mm
- net Net-(U1C--): track 27.6 -> 35.5 mm, vias 3 -> 2
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
Commit message: Casualty 6: pre-order review. RANGE loading fix (RV4 B10k, R43 2k2, Iabc resistors 15k), R53 1M input pulldown; re-routed (DRC 0/0/parity clean); notes
Co-Authored-By: Claude Opus 5.5 <noreply@anthropic.com>
Parts:
- added R53: 1M, Resistor_SMD:R_0805_2012Metric_Pad1.20x1.40mm_HandSolder, F.Cu at (132.2, 139.8)
- R11, R17, R23, R5: value 10k -> 15k
- R43: value 47k -> 2k2
- RV4: value B50k -> B10k
Routing:
- net +9V: track 260.4 -> 207.7 mm, vias 13 -> 7
- net GND: track 362.1 -> 397.3 mm, vias 5 -> 7
- net Net-(SW2B-A): track 78.5 -> 62.3 mm, vias 2 -> 3
- net Net-(SW1B-B): track 52.9 -> 37.8 mm, vias 1 -> 0
- net Net-(SW2A-B): track 34.1 -> 48.7 mm, vias 0 -> 1
- net /DRY: track 79.5 -> 65.7 mm, vias 2 -> 4
- net /PHASE_OUT: track 59.3 -> 72.8 mm, vias 4 -> 2
- net /VREF: track 181.9 -> 169.1 mm
- net /CV: track 71.9 -> 83.2 mm, vias 1 -> 2
- net /X: track 81.5 -> 92.2 mm
- net Net-(U6B--): track 33.5 -> 43.7 mm, vias 2 -> 1
- net /WET: track 14.6 -> 23.6 mm
- net Net-(SW1A-A): track 38.0 -> 46.1 mm
- net Net-(SW2B-B): track 46.3 -> 40.4 mm
- net Net-(U4B--): track 20.9 -> 26.3 mm, vias 2 -> 0
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Other:
- board text added: "SUPER-FREQ after \nCausality 6 by Rick Holt"
- board text removed: "SUPER-FREQ after Causality 6 by Rick Holt"
