File: Casualty6.kicad_sch (KiCad schematic)
At the start: 91 parts, among them J1 9V, J2 G, J3 IN/LED/GND/OUT, J4 IG, J5 OG, SW1 DPDT, SW2 DPDT, U1 LM13700, U2 LM13700, U3 TL072, U4 TL072, U5 TL072, U6 TL072

Commit message: Casualty 6: REGEN fix (U5B non-inverting summer, R48-R50) from ngspice sim; slotted DPDT toggle footprint; full re-route (DRC 0); sim scripts and notes
Co-Authored-By: Claude Opus 5.5 <noreply@anthropic.com>
Parts:
- added R48, R50: 10k, Resistor_SMD:R_0805_2012Metric_Pad1.20x1.40mm_HandSolder, symbol Device:R
- added R49: 6k8, Resistor_SMD:R_0805_2012Metric_Pad1.20x1.40mm_HandSolder, symbol Device:R
Connections:
- net DRY: now also R48.1; no longer C6.1, R27.1, RV6.3
- net REGEN_IN: no longer R30.2
- net VREF: now also R50.2; no longer U5.5 (+)
- net at U5.6 (-): now also R49.1, R50.1; no longer U5.7
- new net REGEN_SUM: R30.2, R48.2, U5.5 (+)
- new net X: C6.1, R27.1, R49.2, RV6.3, U5.7
Other:
- note added: "U5B: REGEN summer, non-inverting x1.68: X = 1.68 (0.6 DRY + 0.4 REGEN). X feeds AP1 and MIX (2026-10-15 sim fix)"
- note removed: "U5B spare (follower, can host a new feature)"

Commit message: Casualty 6: CV IN (J6 + R51 10k) and LFO OUT (J7 + R52 1k) pads; full re-route (DRC 0)
Co-Authored-By: Claude Opus 5.5 <noreply@anthropic.com>
Parts:
- added J6: CV IN, Connector_Wire:SolderWire-0.5sqmm_1x01_D0.9mm_OD2.1mm, symbol Connector_Generic:Conn_01x01
- added J7: LFO OUT, Connector_Wire:SolderWire-0.5sqmm_1x01_D0.9mm_OD2.1mm, symbol Connector_Generic:Conn_01x01
- added R51: 10k, Resistor_SMD:R_0805_2012Metric_Pad1.20x1.40mm_HandSolder, symbol Device:R
- added R52: 1k, Resistor_SMD:R_0805_2012Metric_Pad1.20x1.40mm_HandSolder, symbol Device:R
Connections:
- net CV: now also R51.2
- net at RV3.2, RV3.3, RV4.3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: now also R52.1
- new net: J6.1 (Pin_1), R51.1
- new net LFO_OUT: J7.1 (Pin_1), R52.2
Other:
- note added: "CV IN / LFO OUT (2026-10-15): hooks for a random / S&H LFO or other modulation. Leave unconnected if unused."

Commit message: Casualty 6: pre-order review. RANGE loading fix (RV4 B10k, R43 2k2, Iabc resistors 15k), R53 1M input pulldown; re-routed (DRC 0/0/parity clean); notes
Co-Authored-By: Claude Opus 5.5 <noreply@anthropic.com>
Parts:
- added R53: 1M, Resistor_SMD:R_0805_2012Metric_Pad1.20x1.40mm_HandSolder, symbol Device:R
- R11, R17, R23, R5: value 10k -> 15k; LCSC C17414 -> C17475
- R43: value 47k -> 2k2; LCSC C17713 -> C17520
- RV4: value B50k -> B10k
Connections:
- net GND: now also R53.2
- net IN: now also R53.1
Changed lines of the file:
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@@
 	(wire
 		(pts
-			(xy 538.48 162.56) (xy 541.02 162.56)
+			(xy 538.48 162.56)
+			(xy 541.02 162.56)
 		)
 		(stroke
@@
 	(wire
 		(pts
-			(xy 548.64 162.56) (xy 553.72 162.56)
+			(xy 548.64 162.56)
+			(xy 553.72 162.56)
 		)
 		(stroke
@@
 	(wire
 		(pts
-			(xy 538.48 175.26) (xy 543.56 175.26)
+			(xy 538.48 175.26)
+			(xy 543.56 175.26)
 		)
 		(stroke
@@
 	(wire
 		(pts
-			(xy 223.52 269.24) (xy 223.52 271.78)
+			(xy 223.52 269.24)
+			(xy 223.52 271.78)
 		)
 		(stroke
@@
 	(wire
 		(pts
-			(xy 223.52 279.4) (xy 223.52 281.94)
+			(xy 223.52 279.4)
+			(xy 223.52 281.94)
 		)
 		(stroke
@@
 	(wire
 		(pts
-			(xy 530.86 83.82) (xy 525.78 83.82)
+			(xy 530.86 83.82)
+			(xy 525.78 83.82)
 		)
 		(stroke
@@
 	(wire
 		(pts
-			(xy 525.78 83.82) (xy 525.78 86.36)
+			(xy 525.78 83.82)
+			(xy 525.78 86.36)
 		)
 		(stroke
@@
 	(wire
 		(pts
-			(xy 525.78 93.98) (xy 525.78 96.52)
+			(xy 525.78 93.98)
+			(xy 525.78 96.52)
 		)
 		(stroke
@@
 	(wire
 		(pts
-			(xy 528.32 83.82) (xy 528.32 88.9)
+			(xy 528.32 83.82)
+			(xy 528.32 88.9)
 		)
 		(stroke
@@
 	(wire
 		(pts
-			(xy 528.32 88.9) (xy 535.94 88.9)
+			(xy 528.32 88.9)
+			(xy 535.94 88.9)
 		)
 		(stroke
@@
 	(wire
 		(pts
-			(xy 543.56 88.9) (xy 551.18 88.9)
+			(xy 543.56 88.9)
+			(xy 551.18 88.9)
 		)
 		(stroke
@@
 	(wire
 		(pts
-			(xy 551.18 88.9) (xy 551.18 81.28)
+			(xy 551.18 88.9)
+			(xy 551.18 81.28)
 		)
 		(stroke
@@
 	(wire
 		(pts
-			(xy 551.18 81.28) (xy 556.26 81.28)
+			(xy 551.18 81.28)
+			(xy 556.26 81.28)
 		)
 		(stroke
@@
 	(wire
 		(pts
-			(xy 525.78 78.74) (xy 525.78 73.66)
+			(xy 525.78 78.74)
+			(xy 525.78 73.66)
 		)
 		(stroke
@@
 	(wire
 		(pts
-			(xy 520.7 73.66) (xy 525.78 73.66)
+			(xy 520.7 73.66)
+			(xy 525.78 73.66)
 		)
 		(stroke
@@
 	(wire
 		(pts
-			(xy 510.54 73.66) (xy 513.08 73.66)
+			(xy 510.54 73.66)
+			(xy 513.08 73.66)
 		)
 		(stroke
@@
 			)
 		)
-		(property "Value" "10k"
+		(property "Value" "15k"
 			(at 86.36 66.04 0)
 			(effects
@@
 			)
 		)
-		(property "LCSC" "C17414"
+		(property "LCSC" "C17475"
 			(at 83.82 64.77 0)
 			(hide yes)
@@
 			)
 		)
-		(property "Value" "10k"
+		(property "Value" "15k"
 			(at 162.56 66.04 0)
 			(effects
@@
 			)
 		)
-		(property "LCSC" "C17414"
+		(property "LCSC" "C17475"
 			(at 160.02 64.77 0)
 			(hide yes)
@@
 			)
 		)
-		(property "Value" "10k"
+		(property "Value" "15k"
 			(at 248.92 66.04 0)
 			(effects
@@
 			)
 		)
-		(property "LCSC" "C17414"
+		(property "LCSC" "C17475"
 			(at 246.38 64.77 0)
 			(hide yes)
@@
 			)
 		)
-		(property "Value" "10k"
+		(property "Value" "15k"
 			(at 325.12 66.04 0)
 			(effects
@@
 			)
 		)
-		(property "LCSC" "C17414"
+		(property "LCSC" "C17475"
 			(at 322.58 64.77 0)
 			(hide yes)
@@
 			)
 		)
-		(property "Value" "B50k"
+		(property "Value" "B10k"
 			(at 238.125 280.67 0)
 			(effects
@@
 			)
 		)
-		(property "Description" "RANGE pot, 16mm, hand-soldered"
+		(property "Description" "RANGE (B10k: even sweep with R43 2k2 and 15k per OTA)"
 			(at 233.68 279.4 0)
 			(hide yes)
@@
 			)
 		)
-		(property "Value" "47k"
+		(property "Value" "2k2"
 			(at 231.14 288.29 0)
 			(effects
@@
 			)
 		)
-		(property "Description" "RANGE bottom (original R8)"
+		(property "Description" "RANGE bottom (was 47k)"
 			(at 233.68 287.02 0)
 			(hide yes)
@@
 			)
 		)
-		(property "LCSC" "C17713"
+		(property "LCSC" "C17520"
 			(at 233.68 287.02 0)
 			(hide yes)
@@
 					(unit 1)
 				)
+			)
+		)
+	)
+	(junction
+		(at 22.86 147.32)
+		(diameter 0)
+		(color 0 0 0 0)
+	)
+	(symbol
+		(lib_id "Device:R")
+		(at 22.86 151.13 0)
+		(unit 1)
+		(exclude_from_sim no)
+		(in_bom yes)
+		(on_board yes)
+		(dnp no)
+		(property "Reference" "R53"
+			(at 20.32 149.86 0)
+			(effects
+				(font
+					(size 1.27 1.27)
+				)
+				(justify right)
+			)
+		)
+		(property "Value" "1M"
+			(at 20.32 152.4 0)
+			(effects
+				(font
+					(size 1.27 1.27)
+				)
+				(justify right)
+			)
+		)
+		(property "Footprint" "Resistor_SMD:R_0805_2012Metric_Pad1.20x1.40mm_HandSolder"
+			(at 22.86 151.13 0)
+			(hide yes)
+			(effects
+				(font
+					(size 1.27 1.27)
+				)
+			)
+		)
+		(property "Datasheet" ""
+			(at 22.86 151.13 0)
+			(hide yes)
+			(effects
+				(font
+					(size 1.27 1.27)
+				)
+			)
+		)
+		(property "Description" "Input pulldown (no pop when switching in)"
+			(at 22.86 151.13 0)
+			(hide yes)
+			(effects
+				(font
+					(size 1.27 1.27)
+				)
+			)
+		)
+		(property "LCSC" "C17514"
+			(at 22.86 151.13 0)
+			(hide yes)
+			(effects
+				(font
+					(size 1.27 1.27)
+				)
+			)
+		)
+		(pin "1"
+		)
+		(pin "2"
+		)
+		(instances
+			(project "Casualty6"
+				(path "/ddad1137-1dd8-4722-992e-184d1837bd0a"
+					(reference "R53")
+					(unit 1)
+				)
+			)
+		)
+	)
+	(symbol
+		(lib_id "power:GND")
+		(at 22.86 154.94 0)
+		(unit 1)
+		(exclude_from_sim no)
+		(in_bom yes)
+		(on_board yes)
+		(dnp no)
+		(property "Reference" "#PWR401"
+			(at 22.86 154.94 0)
+			(hide yes)
+			(effects
+				(font
+					(size 1.27 1.27)
+				)
+			)
+		)
+		(property "Value" "GND"
+			(at 22.86 158.75 0)
+			(effects
+				(font
+					(size 1.27 1.27)
+				)
+			)
+		)
+		(property "Footprint" ""
+			(at 22.86 154.94 0)
+			(hide yes)
+			(effects
+				(font
+					(size 1.27 1.27)
+				)
+			)
+		)
+		(property "Datasheet" ""
+			(at 22.86 154.94 0)
+			(hide yes)
+			(effects
+				(font
+					(size 1.27 1.27)
+				)
+			)
+		)
+		(property "Description" ""
+			(at 22.86 154.94 0)
+			(hide yes)
+			(effects
+				(font
+					(size 1.27 1.27)
+				)
+			)
+		)
+		(pin "1"
+		)
+		(instances
+			(project "Casualty6"
+				(path "/ddad1137-1dd8-4722-992e-184d1837bd0a"
+					(reference "#PWR401")
+					(unit 1)
+				)

Commit message: U1-U6: FT Rotation Offset 270 (JLC preview needed 90 CW on 2 of 3 web uploads); order notes updated
Co-Authored-By: Claude Opus 5.5 <noreply@anthropic.com>
Parts:
- U1, U2, U3, U4, U5, U6: FT Rotation Offset (none) -> 270
Changed lines of the file:
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@@
 			)
 		)
+		(property "FT Rotation Offset" "270"
+			(at 76.2 50.8 0)
+			(hide yes)
+			(effects
+				(font
+					(size 1.27 1.27)
+				)
+			)
+		)
 		(pin "1"
 		)
@@
 			)
 		)
+		(property "FT Rotation Offset" "270"
+			(at 101.6 50.8 0)
+			(hide yes)
+			(effects
+				(font
+					(size 1.27 1.27)
+				)
+			)
+		)
 		(pin "7"
 		)
@@
 			)
 		)
+		(property "FT Rotation Offset" "270"
+			(at 152.4 50.8 0)
+			(hide yes)
+			(effects
+				(font
+					(size 1.27 1.27)
+				)
+			)
+		)
 		(pin "12"
 		)
@@
 			)
 		)
+		(property "FT Rotation Offset" "270"
+			(at 177.8 50.8 0)
+			(hide yes)
+			(effects
+				(font
+					(size 1.27 1.27)
+				)
+			)
+		)
 		(pin "9"
 		)
@@
 			)
 		)
+		(property "FT Rotation Offset" "270"
+			(at 238.76 50.8 0)
+			(hide yes)
+			(effects
+				(font
+					(size 1.27 1.27)
+				)
+			)
+		)
 		(pin "1"
 		)
@@
 			)
 		)
+		(property "FT Rotation Offset" "270"
+			(at 264.16 50.8 0)
+			(hide yes)
+			(effects
+				(font
+					(size 1.27 1.27)
+				)
+			)
+		)
 		(pin "7"
 		)
@@
 			)
 		)
+		(property "FT Rotation Offset" "270"
+			(at 314.96 50.8 0)
+			(hide yes)
+			(effects
+				(font
+					(size 1.27 1.27)
+				)
+			)
+		)
 		(pin "12"
 		)
@@
 			)
 		)
+		(property "FT Rotation Offset" "270"
+			(at 340.36 50.8 0)
+			(hide yes)
+			(effects
+				(font
+					(size 1.27 1.27)
+				)
+			)
+		)
 		(pin "9"
 		)
@@
 			)
 		)
+		(property "FT Rotation Offset" "270"
+			(at 68.58 149.86 0)
+			(hide yes)
+			(effects
+				(font
+					(size 1.27 1.27)
+				)
+			)
+		)
 		(pin "1"
 		)
@@
 			)
 		)
+		(property "FT Rotation Offset" "270"
+			(at 68.58 187.96 0)
+			(hide yes)
+			(effects
+				(font
+					(size 1.27 1.27)
+				)
+			)
+		)
 		(pin "5"
 		)
@@
 			)
 		)
+		(property "FT Rotation Offset" "270"
+			(at 251.46 147.32 0)
+			(hide yes)
+			(effects
+				(font
+					(size 1.27 1.27)
+				)
+			)
+		)
 		(pin "1"
 		)
@@
 			)
 		)
+		(property "FT Rotation Offset" "270"
+			(at 264.16 187.96 0)
+			(hide yes)
+			(effects
+				(font
+					(size 1.27 1.27)
+				)
+			)
+		)
 		(pin "5"
 		)
@@
 			)
 		)
+		(property "FT Rotation Offset" "270"
+			(at 60.96 269.24 0)
+			(hide yes)
+			(effects
+				(font
+					(size 1.27 1.27)
+				)
+			)
+		)
 		(pin "1"
 		)
@@
 			)
 		)
+		(property "FT Rotation Offset" "270"
+			(at 198.12 269.24 0)
+			(hide yes)
+			(effects
+				(font
+					(size 1.27 1.27)
+				)
+			)
+		)
 		(pin "5"
 		)
@@
 			)
 		)
+		(property "FT Rotation Offset" "270"
+			(at 538.48 48.26 0)
+			(hide yes)
+			(effects
+				(font
+					(size 1.27 1.27)
+				)
+			)
+		)
 		(pin "1"
 		)
@@
 			)
 		)
+		(property "FT Rotation Offset" "270"
+			(at 538.48 81.28 0)
+			(hide yes)
+			(effects
+				(font
+					(size 1.27 1.27)
+				)
+			)
+		)
 		(pin "5"
 		)
@@
 			)
 		)
+		(property "FT Rotation Offset" "270"
+			(at 403.86 121.92 0)
+			(hide yes)
+			(effects
+				(font
+					(size 1.27 1.27)
+				)
+			)
+		)
 		(pin "6"
 		)
@@
 			)
 		)
+		(property "FT Rotation Offset" "270"
+			(at 429.26 121.92 0)
+			(hide yes)
+			(effects
+				(font
+					(size 1.27 1.27)
+				)
+			)
+		)
 		(pin "6"
 		)
@@
 			)
 		)
+		(property "FT Rotation Offset" "270"
+			(at 454.66 121.92 0)
+			(hide yes)
+			(effects
+				(font
+					(size 1.27 1.27)
+				)
+			)
+		)
 		(pin "4"
 		)
@@
 			)
 		)
+		(property "FT Rotation Offset" "270"
+			(at 480.06 121.92 0)
+			(hide yes)
+			(effects
+				(font
+					(size 1.27 1.27)
+				)
+			)
+		)
 		(pin "4"
 		)
@@
 			)
 		)
+		(property "FT Rotation Offset" "270"
+			(at 505.46 121.92 0)
+			(hide yes)
+			(effects
+				(font
+					(size 1.27 1.27)
+				)
+			)
+		)
 		(pin "4"
 		)
@@
 			(at 530.86 121.92 0)
 			(hide yes)
+			(effects
+				(font
+					(size 1.27 1.27)
+				)
+			)
+		)
+		(property "FT Rotation Offset" "270"
+			(at 530.86 121.92 0)
+			(hide yes)
